File: ECU_Hardware/stm32_ecu.kicad_pcb (KiCad board)
At the start: 2 copper layers, 62 parts, among them J1 TC2030-NL, J2 USB_C_Receptacle_USB2.0_16P, U1 ATGM336H-5N31, U11 STM32G474CEUx, U20 USBLC6-2P6, U6 AP2112K-3.3

Commit message: Move ECU schematics into schematics/ and add driver inputs and sensor notes
Hierarchical sheets now live in ECU_Hardware/schematics, with the new
Driver_Inputs sheet (APPS, BPPS and steering dividers and clamps), the
reviewed and JLCPCB project symbol libraries, new 3D models, and
SENSOR_INTERFACES.md with the GPS, IMU and temperature pin allocation.
The old top-level sheets and the restore backup are removed.

Claude-Session: https://claude.ai/code/session_0117trEbCv7z6CPYkN3K3GKQ
Parts:
- added C100: 10uF, PCM_JLCPCB:C_0603, F.Cu at (169.3, 57.6)
- added C101: 100nF, PCM_JLCPCB:C_0603, F.Cu at (169.3, 59.9)
- added C102: 100nF, PCM_JLCPCB:C_0603, F.Cu at (169.3, 62.1)
- added C11: 100nF, PCM_JLCPCB:C_0402, F.Cu at (163.9, 61.1)
- added C110: 10nF, PCM_JLCPCB:C_0603, F.Cu at (136.7, 33.8)
- added C111: 10nF, PCM_JLCPCB:C_0603, F.Cu at (136.7, 36.1)
- added C112: 10nF, PCM_JLCPCB:C_0603, F.Cu at (136.7, 38.3)
- added C113: 10nF, PCM_JLCPCB:C_0603, F.Cu at (136.7, 40.6)
- added C120: 100nF, PCM_JLCPCB:C_0603, F.Cu at (159.2, 42.1)
- added C121: 100nF, PCM_JLCPCB:C_0603, F.Cu at (159.2, 44.4)
- added C122: 100nF, PCM_JLCPCB:C_0603, F.Cu at (159.2, 46.6)
- added C123: 22uF, PCM_JLCPCB:C_0603, F.Cu at (160.0, 35.5)
- added C124: 100nF, PCM_JLCPCB:C_0603, F.Cu at (160.0, 37.7)
- added C7: 1uF, PCM_JLCPCB:C_0402, F.Cu at (163.9, 57.4)
- added C8: 100nF, PCM_JLCPCB:C_0402, F.Cu at (168.8, 68.6)
- added C9: 100nF, PCM_JLCPCB:C_0402, F.Cu at (163.9, 59.3)
- added CN1: XT60PW-M, easyeda2kicad:CONN-TH_XT60PW-M, F.Cu at (185.3, 61.9)
- added CN2: XDWF-C3030WR-2*3P, easyeda2kicad:CONN-TH_XDWF-C3030WR-2X3P, F.Cu at (188.2, 45.0)
- added CN3: XDWF-C3030WR-2*3P, easyeda2kicad:CONN-TH_XDWF-C3030WR-2X3P, F.Cu at (188.1, 31.4)
- added CN4: XDWF-C3030WR-2*3P, easyeda2kicad:CONN-TH_XDWF-C3030WR-2X3P, F.Cu at (188.2, 18.0)
- added D110: BAT54S, Package_TO_SOT_SMD:SOT-23, F.Cu at (132.4, 25.9)
- added D111: BAT54S, Package_TO_SOT_SMD:SOT-23, F.Cu at (132.4, 30.4)
- added D112: BAT54S, Package_TO_SOT_SMD:SOT-23, F.Cu at (132.4, 34.8)
- added D113: BAT54S, Package_TO_SOT_SMD:SOT-23, F.Cu at (132.4, 39.3)
- added D114: BAT54S, Package_TO_SOT_SMD:SOT-23, F.Cu at (160.5, 32.1)
- added D15: White, PCM_JLCPCB:D_0805, F.Cu at (150.0, 34.5)
- added J3: U.FL, PCM_JLCPCB:IPEX-SMD_BWIPX-1-001E, F.Cu at (173.0, 59.0)
- added L2: SWPA5040S150MT, easyeda2kicad:IND-SMD_L5.0-W5.0, F.Cu at (158.0, 26.8)
- added L3: ACT45B-101-2P-TL003, easyeda2kicad:FILTER-SMD_4P-L4.5-W3.2-TL_ACT45B, F.Cu at (151.2, 43.8)
- added L4: 47nH, PCM_JLCPCB:L_0402, F.Cu at (172.6, 62.5)
- added R1: 220kΩ, PCM_JLCPCB:R_0603, F.Cu at (156.3, 31.0)
- added R110: 33kΩ, PCM_JLCPCB:R_0603, F.Cu at (136.6, 24.8)
- added R111: 47kΩ, PCM_JLCPCB:R_0603, F.Cu at (136.6, 27.1)
- added R112: 1kΩ, PCM_JLCPCB:R_0603, F.Cu at (136.6, 29.3)
- added R113: 33kΩ, PCM_JLCPCB:R_0603, F.Cu at (136.6, 31.6)
- added R114: 47kΩ, PCM_JLCPCB:R_0603, F.Cu at (140.3, 24.8)
- added R115: 1kΩ, PCM_JLCPCB:R_0603, F.Cu at (140.3, 27.1)
- added R116: 33kΩ, PCM_JLCPCB:R_0603, F.Cu at (140.3, 29.3)
- added R117: 47kΩ, PCM_JLCPCB:R_0603, F.Cu at (140.3, 31.6)
- added R118: 1kΩ, PCM_JLCPCB:R_0603, F.Cu at (143.9, 24.8)
- added R119: 33kΩ, PCM_JLCPCB:R_0603, F.Cu at (143.9, 27.1)
- added R120: 47kΩ, PCM_JLCPCB:R_0603, F.Cu at (143.9, 29.3)
- added R121: 1kΩ, PCM_JLCPCB:R_0603, F.Cu at (143.9, 31.6)
- added R130: 1kΩ, PCM_JLCPCB:R_0603, F.Cu at (156.3, 35.5)
- added R2: 10kΩ, PCM_JLCPCB:R_0402, F.Cu at (163.9, 63.0)
- added R3: 39kΩ, PCM_JLCPCB:R_0402, F.Cu at (168.8, 70.4)
- added R4: 10kΩ, PCM_JLCPCB:R_0603, F.Cu at (156.3, 33.3)
- added R5: 10kΩ, PCM_JLCPCB:R_0402, F.Cu at (153.9, 46.9)
- added TH1: 10k NTC, PCM_JLCPCB:R_0603, F.Cu at (169.2, 66.5)
- added U2: LMR38020SQDDARQ1, easyeda2kicad:SOIC-8_L4.9-W3.9-P1.27-LS6.0-BL-EP3.4, F.Cu at (151.3, 28.3)
- added U3: LSM6DSV16XTR, easyeda2kicad:LGA-14_L3.0-W2.5-P0.50-BR, F.Cu at (155.7, 90.4)
- added U4: TCAN337GDCNR, easyeda2kicad:SOT-23-8_L3.0-W1.7-P0.65-LS2.8-BR, F.Cu at (150.1, 48.1)
- added U5: LM66200DRLR, easyeda2kicad:SOT-583-8_L2.1-W1.2-P0.50-LS1.6-BL, F.Cu at (149.6, 37.5)
- added U7: XD-43045-2*2AW, easyeda2kicad:CONN-TH_4P-P3.00_XUNDA_XD-43045-2_2AW, F.Cu at (188.3, 87.5)
- added U8: XD-43045-2*2AW, easyeda2kicad:CONN-TH_4P-P3.00_XUNDA_XD-43045-2_2AW, F.Cu at (188.3, 76.6)
- added X1: XC7EL89COO-114YLC-16M, easyeda2kicad:CRYSTAL-SMD_4P-L2.0-W1.6-BL, F.Cu at (132.1, 45.4)
- C58, C79: value 4.7uF -> 22uF
- FB3: value ~ -> 120Ω @100MHz
- R64, R65: value 60Ω -> 60.4Ω
Connections:
- U1 pad 1: unconnected-(U1-GND-Pad1) -> GND
- U1 pad 10: unconnected-(U1-GND-Pad10) -> GND
- U1 pad 11: unconnected-(U1-RF_IN-Pad11) -> Net-(J3-In)
- U1 pad 12: unconnected-(U1-GND-Pad12) -> GND
- U1 pad 14: unconnected-(U1-VCC_RF-Pad14) -> /GPS/GPS_ANT_BIAS
- U1 pad 2: unconnected-(U1-TXD-Pad2) -> /GPS_RX
- U1 pad 3: unconnected-(U1-RXD-Pad3) -> /GPS_TX
- U1 pad 4: unconnected-(U1-1PPS-Pad4) -> /GPS_PPS
- U1 pad 6: unconnected-(U1-VBAT-Pad6) -> +3V3
- U1 pad 8: unconnected-(U1-VCC-Pad8) -> +3V3
- U11 pad 10: unconnected-(U11-PA2-Pad10) -> /APPS_2
- U11 pad 11: unconnected-(U11-PA3-Pad11) -> /BPPS
- U11 pad 12: unconnected-(U11-PA4-Pad12) -> /IMU_CS_N
- U11 pad 13: unconnected-(U11-PA5-Pad13) -> /IMU_SCK
- U11 pad 14: unconnected-(U11-PA6-Pad14) -> /IMU_MISO
- U11 pad 15: unconnected-(U11-PA7-Pad15) -> /IMU_MOSI
- U11 pad 16: unconnected-(U11-PC4-Pad16) -> /IMU_INT
- U11 pad 17: unconnected-(U11-PB0-Pad17) -> /STEERING
- U11 pad 18: unconnected-(U11-PB1-Pad18) -> /VIN_SENSE
- U11 pad 30: unconnected-(U11-PA8-Pad30) -> /GPS_PPS
- U11 pad 31: unconnected-(U11-PA9-Pad31) -> /GPS_TX
- U11 pad 32: unconnected-(U11-PA10-Pad32) -> /GPS_RX
- U11 pad 8: unconnected-(U11-PA0-Pad8) -> /TEMP_SENSE
- U11 pad 9: unconnected-(U11-PA1-Pad9) -> /APPS_1
