File: ECU_Hardware/schematics/CAN.kicad_sch (KiCad schematic)
At the start: 11 parts, among them U4 TCAN337GDCNR

Commit message: Move ECU schematics into schematics/ and add driver inputs and sensor notes
Hierarchical sheets now live in ECU_Hardware/schematics, with the new
Driver_Inputs sheet (APPS, BPPS and steering dividers and clamps), the
reviewed and JLCPCB project symbol libraries, new 3D models, and
SENSOR_INTERFACES.md with the GPS, IMU and temperature pin allocation.
The old top-level sheets and the restore backup are removed.

Claude-Session: https://claude.ai/code/session_0117trEbCv7z6CPYkN3K3GKQ
Parts:
- removed R64, R65: 60Ω, PCM_JLCPCB:R_0603, symbol PCM_JLCPCB-Resistors:0603,33Ω
- added R1, R4: 60.4Ω, PCM_JLCPCB:R_0402, symbol PCM_JLCPCB-Resistors:0402,10kΩ
- added R5: 10kΩ, PCM_JLCPCB:R_0402, symbol PCM_JLCPCB-Resistors:0402,10kΩ
- D9: symbol can:ESDCAN03-2BWY -> ECU_Reviewed:ESDCAN03-2BWY
- L3: symbol easyeda2kicad:ACT45B-101-2P-TL003 -> ECU_Reviewed:ACT45B-101-2P-TL003
- U4: symbol easyeda2kicad:TCAN337GDCNR -> ECU_Reviewed:TCAN337GDCNR
Connections:
- net +3V3: now also R5.2
- net CAN_FAULT: now also R5.1
- net CAN_UNFIL_N: now also R1.1
- net CAN_UNFIL_P: now also R4.1
- net GND: now also U4.8 (S)
- net at C5.2: now also R1.2, R4.2
- no-connect marks 1 -> 0
Other:
- note added: "JP1 + JP2 OPEN: intermediate node (default). Bridge BOTH only at a physical bus end: 120.8 ohm split termination. CAN_FAULT is HIGH on fault; R131 provides the required pull-up. S tied low: normal operation. Check CAN-FD waveform with selected choke/caps."
