File: ECU_Hardware/schematics/Connectors.kicad_sch (KiCad schematic)
At the start: 8 parts, among them J1 TC2030-NL, J2 USB_C_Receptacle_USB2.0_16P, U20 USBLC6-2P6

Commit message: Move ECU schematics into schematics/ and add driver inputs and sensor notes
Hierarchical sheets now live in ECU_Hardware/schematics, with the new
Driver_Inputs sheet (APPS, BPPS and steering dividers and clamps), the
reviewed and JLCPCB project symbol libraries, new 3D models, and
SENSOR_INTERFACES.md with the GPS, IMU and temperature pin allocation.
The old top-level sheets and the restore backup are removed.

Claude-Session: https://claude.ai/code/session_0117trEbCv7z6CPYkN3K3GKQ
Parts:
- added CN1: XT60PW-M, easyeda2kicad:CONN-TH_XT60PW-M, symbol ECU_Reviewed:XT60PW-M
- added CN2, CN3, CN5: XDWF-C3030WR-2*3P, easyeda2kicad:CONN-TH_XDWF-C3030WR-2X3P, symbol ECU_Reviewed:XDWF-C3030WR-2*3P
- added U7, U8: XD-43045-2*2AW, easyeda2kicad:CONN-TH_4P-P3.00_XUNDA_XD-43045-2_2AW, symbol ECU_Reviewed:XD-43045-2*2AW
- FB3: value (none) -> 120Ω @100MHz
- J2: symbol Connector:USB_C_Receptacle_USB2.0_16P -> ECU_Reviewed:USB_C_Receptacle_USB2.0_16P
- U20: symbol Power_Protection:USBLC6-2P6 -> ECU_Reviewed:USBLC6-2P6
Connections:
- net CAN_UNFIL_N: now also U7.2, U8.2
- net CAN_UNFIL_P: now also U7.1, U8.1
- net GND: now also CN1.1 (-), CN1.3, CN1.4, CN2.2, CN2.5, CN3.2, CN3.5, CN5.2, CN5.5, U7.3, U8.3
- net VIN_12_60V: now also CN1.2 (+)
- new net 5V_OR: CN2.1, CN2.4, CN3.1, CN3.4, CN5.1, CN5.4
- new net APPS_1_RAW: CN2.3
- new net APPS_2_RAW: CN2.6
- new net BPPS_RAW: CN3.3
- new net STEERING_RAW: CN5.3
- no-connect marks 2 -> 6
Other:
- note added: "Accelerator Pedal Position Sensor"
- note added: "Board Power Connector"
- note added: "Brake Pedal Position Sensor"
- note added: "CAN"
- note added: "Steering Angle Sensor"
- note removed: "CAN Connector"
- note removed: "TBD"
- note removed: "TBD: XT60 + protection, two parallel CAN connectors, pedal/steering connectors and input conditioning. Sensor supply is +5V_BUCK (before ORing), never USB/5V_OR."
