File: ECU_Hardware/schematics/MCU.kicad_sch (KiCad schematic)
At the start: 24 parts, among them U11 STM32G474CEUx, X1 XC7EL89COO-114YLC-16M

Commit message: Move ECU schematics into schematics/ and add driver inputs and sensor notes
Hierarchical sheets now live in ECU_Hardware/schematics, with the new
Driver_Inputs sheet (APPS, BPPS and steering dividers and clamps), the
reviewed and JLCPCB project symbol libraries, new 3D models, and
SENSOR_INTERFACES.md with the GPS, IMU and temperature pin allocation.
The old top-level sheets and the restore backup are removed.

Claude-Session: https://claude.ai/code/session_0117trEbCv7z6CPYkN3K3GKQ
Parts:
- S1, S2: symbol PCM_JLCPCB-Connectors_Buttons:Tactile Button, 160gf, 12V, 50mA, 4.0mm -> ECU_Reviewed:Tactile Button, 160gf, 12V, 50mA, 4.0mm
- X1: symbol easyeda2kicad:XC7EL89COO-114YLC-16M -> ECU_Reviewed:XC7EL89COO-114YLC-16M
Connections:
- net APPS_1: now also U11.9 (PA1)
- net APPS_2: now also U11.10 (PA2)
- net BPPS: now also U11.11 (PA3)
- net GPS_PPS: now also U11.30 (PA8)
- net GPS_RX: now also U11.32 (PA10)
- net GPS_TX: now also U11.31 (PA9)
- net IMU_CS_N: now also U11.12 (PA4)
- net IMU_INT: now also U11.16 (PC4)
- net IMU_MISO: now also U11.14 (PA6)
- net IMU_MOSI: now also U11.15 (PA7)
- net IMU_SCK: now also U11.13 (PA5)
- net STEERING: now also U11.17 (PB0)
- net VIN_SENSE: now also U11.18 (PB1)
- net TEMP_SENSE: now reaches U11.8 (PA0)
- no-connect marks 29 -> 15
Other:
- note added: "ADC1: PA0 temp; PA1 APPS1; PA2 APPS2; PA3 brake; PB0 steering; PB1 VIN. Configure analog / no pulls; long acquisition time; reject implausible or stale inputs. VIN = ADC voltage x23. Require main input present before issuing torque commands. USART1 AF7: PA9 TX / PA10 RX; PPS PA8 TIM1_CH1 AF6. SPI1 AF5: PA5/6/7; PA4 CS; PC4 EXTI4. FDCAN2 AF9: PB5 RX / PB6 TX. Receiving motor controllers must time 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"
- note removed: "RESERVED INTERFACES - MCU GPIO/ADC/AF allocation TBD. These ports are not yet wired to MCU pins. Heartbeat LED is local."
- note removed: "TBD"
